File: hw-proto01/hw-proto01.sch (EAGLE design)
At the start: 4 parts, among them Q1 PMOS, Q2 PMOS

Commit message: initial eagle drawings
Parts:
- removed R1, R2: (no value), rcl:R-US_R0805
- added CAN: (no value), con-amp-quick:M03
- added IC1, IC2: VN5E160MSTR-E, VN5E160MSTR-E:VN5E160MSTR-E
- added IC3: MCP2562T-H_SN, MCP2562T-H_SN:MCP2562T-H_SN
- added IC4: ESP32-WROOM-32E-N8R2, ESP32-WROOM-32E-N8R2:ESP32-WROOM-32E-N8R2
- added PWR: 4DB-P108-06, 4DB-P108-06:4DB-P108-06
Connections:
- new net GND: IC1.GND, IC2.GND, IC3.VDD, IC4.GND_1, IC4.GND_10, IC4.GND_11, IC4.GND_12, IC4.GND_2, IC4.GND_3, IC4.GND_4, IC4.GND_5, IC4.GND_6, IC4.GND_7, IC4.GND_8, IC4.GND_9, PWR.2, PWR.4, PWR.6
- new net N$1: CAN.1, IC3.CANH
- new net N$2: CAN.3, IC3.CANL
- new net SW1: PWR.3, Q1.D
- new net SW2: PWR.5, Q2.D
- net GATE1D: now also IC1.OUT_1, IC1.OUT_2; no longer R1.1
- net GATE2D: now also IC2.OUT_1, IC2.OUT_2; no longer R2.1
- net VPP: now also PWR.1; no longer R1.2, R2.2

Commit message: initial drawings
Parts:
- added PS1: TSR_1-2433E, TSR_1-2433E:TSR_1-2433E
Connections:
- new net +3V3: IC3.VSS, IC4.3V3, PS1.VOUT+
- net GND: now also PS1.GND
- net VPP: now also PS1.VIN+
Changed lines of the file:
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@@
 <part name="SUPPLY2" library="supply2" deviceset="VPP" device=""/>
 <part name="GND6" library="supply1" deviceset="GND" device=""/>
+<part name="PS1" library="TSR_1-2433E" deviceset="TSR_1-2433E" device=""/>
+<part name="SUPPLY3" library="supply2" deviceset="VPP" device=""/>
+<part name="GND7" library="supply1" deviceset="GND" device=""/>
+<part name="+3V1" library="supply1" deviceset="+3V3" device=""/>
+<part name="+3V2" library="supply1" deviceset="+3V3" device=""/>
+<part name="+3V3" library="supply1" deviceset="+3V3" device=""/>
 </parts>
 <sheets>
@@
 <instance part="SUPPLY2" gate="G$1" x="132.08" y="109.22"/>
 <instance part="GND6" gate="1" x="78.74" y="185.42"/>
+<instance part="PS1" gate="G$1" x="165.1" y="144.78" rot="R90"/>
+<instance part="SUPPLY3" gate="G$1" x="144.78" y="154.94"/>
+<instance part="GND7" gate="1" x="167.64" y="127"/>
+<instance part="+3V1" gate="G$1" x="193.04" y="157.48"/>
+<instance part="+3V2" gate="G$1" x="-50.8" y="241.3"/>
+<instance part="+3V3" gate="G$1" x="78.74" y="231.14"/>
 </instances>
 <busses>
@@
 <wire x1="147.32" y1="99.06" x2="132.08" y2="99.06" width="0.1524" layer="91"/>
 <wire x1="132.08" y1="99.06" x2="132.08" y2="106.68" width="0.1524" layer="91"/>
+</segment>
+<segment>
+<pinref part="SUPPLY3" gate="G$1" pin="VPP"/>
+<wire x1="144.78" y1="152.4" x2="144.78" y2="142.24" width="0.1524" layer="91"/>
+<pinref part="PS1" gate="G$1" pin="VIN+"/>
+<wire x1="144.78" y1="142.24" x2="165.1" y2="142.24" width="0.1524" layer="91"/>
+<wire x1="165.1" y1="142.24" x2="165.1" y2="144.78" width="0.1524" layer="91"/>
 </segment>
 </net>
@@
 <wire x1="78.74" y1="210.82" x2="78.74" y2="187.96" width="0.1524" layer="91"/>
 </segment>
+<segment>
+<pinref part="PS1" gate="G$1" pin="GND"/>
+<pinref part="GND7" gate="1" pin="GND"/>
+<wire x1="167.64" y1="144.78" x2="167.64" y2="129.54" width="0.1524" layer="91"/>
+</segment>
 </net>
 <net name="SW1" class="0">
@@
 </segment>
 </net>
+<net name="+3V3" class="0">
+<segment>
+<pinref part="PS1" gate="G$1" pin="VOUT+"/>
+<wire x1="170.18" y1="144.78" x2="170.18" y2="142.24" width="0.1524" layer="91"/>
+<pinref part="+3V1" gate="G$1" pin="+3V3"/>
+<wire x1="170.18" y1="142.24" x2="193.04" y2="142.24" width="0.1524" layer="91"/>
+<wire x1="193.04" y1="142.24" x2="193.04" y2="154.94" width="0.1524" layer="91"/>
+</segment>
+<segment>
+<pinref part="IC4" gate="G$1" pin="3V3"/>
+<pinref part="+3V2" gate="G$1" pin="+3V3"/>
+<wire x1="-5.08" y1="223.52" x2="-50.8" y2="223.52" width="0.1524" layer="91"/>
+<wire x1="-50.8" y1="223.52" x2="-50.8" y2="238.76" width="0.1524" layer="91"/>
+</segment>
+<segment>
+<pinref part="IC3" gate="G$1" pin="VSS"/>
+<pinref part="+3V3" gate="G$1" pin="+3V3"/>
+<wire x1="96.52" y1="213.36" x2="78.74" y2="213.36" width="0.1524" layer="91"/>
+<wire x1="78.74" y1="213.36" x2="78.74" y2="228.6" width="0.1524" layer="91"/>
+</segment>
+</net>

Commit message: initial layout and routing
Parts:
- added C1, C2: 100n, rcl:C-USC0603K
- added IC5: IR4427S, ir:IR4427S
- added J1, J2: 000, rcl:R-US_0207/12
- added R1, R2: 10K0, rcl:R-US_0204/7
- added VREG1: +5V, TSR_1-2433E:TSR_1-2433E
- CAN: device con-amp-quick:M03 -> con-wago-500:W237-103
- MCU: value ESP32-WROOM-32E-N8R2 -> ESP32-WROOM-32E
- VREG2: value TSR_1-2433E -> +3V3
- renumbered IC4 to MCU, PS1 to VREG2
Connections:
- removed net GATE1D: IC1.OUT_1, IC1.OUT_2, Q1.G
- removed net GATE2D: IC2.OUT_1, IC2.OUT_2, Q2.G
- removed net VPP: PWR.1, Q1.S, Q2.S, VREG2.VIN+
- new net +12V: IC1.VCC_1, IC1.VCC_2, IC2.VCC_1, IC2.VCC_2, IC5.VS, PWR.1, Q1.S, Q2.S, VREG1.VIN+, VREG2.VIN+
- new net +5V: C1.1, IC3.VDD, VREG1.VOUT+
- new net CAN_RX: IC3.RXD, MCU.IO21
- new net CAN_TX: IC3.TXD, MCU.IO22
- new net CTL1: IC5.INA, MCU.IO16
- new net CTL2: IC5.INB, MCU.IO17
- new net CTL3: MCU.IO12, R1.1
- new net CTL4: MCU.IO14, R2.1
- new net N$3: IC5.OUTB, J2.1
- new net N$4: IC5.OUTA, J1.1
- new net N$5: J1.2, Q1.G
- new net N$6: J2.2, Q2.G
- new net N$7: IC1.IN, R1.2
- new net N$8: IC2.IN, R2.2
- new net SW3: IC1.OUT_1, IC1.OUT_2, PWR.5
- new net SW4: IC2.OUT_1, IC2.OUT_2, PWR.6
- net +3V3: now also C2.1, IC3.VIO; no longer IC3.VSS
- net GND: now also C1.2, C2.2, IC3.VSS, IC5.GND, VREG1.GND; no longer IC3.VDD, PWR.4, PWR.6
- net N$1: now also CAN-3.KL; no longer CAN.1
- net N$2: now also CAN-1.KL; no longer CAN.3
- net SW2: now also PWR.4; no longer PWR.5
Other:
- moved on the sheet: IC1, IC2, Q2

Commit message: layout refinement, adding passives
Parts:
- added PROG: 1X5, adafruit:1X5
- added R3, R4, R5, R6, R7: 47K0, rcl:R-US_R0603
- IC3: value MCP2562T-H_SN -> MCP2562T
- renumbered VREG1 to VR5V0, VREG2 to VR3V3
Connections:
- new net EN: MCU.EN, PROG.3
- new net GPIO0: MCU.IO0, PROG.4, R4.2
- new net GPIO12: MCU.IO12, R5.1
- new net GPIO15: MCU.IO15, R3.2
- new net GPIO2: MCU.IO2, R6.1
- new net GPIO5: MCU.IO5, R7.2
- new net RXD0: MCU.RXD0, PROG.2
- new net TXD0: MCU.TXD0, PROG.1
- net +3V3: now also R3.1, R4.1, R7.1
- net CTL1: now also MCU.IO18; no longer MCU.IO16
- net CTL2: now also MCU.IO19; no longer MCU.IO17
- net CTL3: now also MCU.IO27; no longer MCU.IO12
- net CTL4: now also MCU.IO26; no longer MCU.IO14
- net GND: now also PROG.5, R5.2, R6.2
