File: hw-proto04/hw-proto04.sch (EAGLE design)
At the start: 34 parts, among them IC1 VN5E160MSTR-E, IC2 UCC27523DR, IC3 MCP2562T, IC4 STM32F042C6T7, IC5 TLV74333PDBVR, J1 10, J2 10, Q1 SQJ147ELP-T1_GE3, Q2 SQJ147ELP-T1_GE3

Commit message: added term resistor, layout refinement
Parts:
- added RTERM: 120R, rcl:R-US_R0805
Connections:
- net CANH: now also RTERM.2
- net CANL: now also RTERM.1
Changed lines of the file:
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@@
 <part name="RDIV2" library="rcl" deviceset="R-US_" device="R0805"/>
 <part name="RBOOT0" library="rcl" deviceset="R-US_" device="R0603" value="100K"/>
+<part name="RTERM" library="rcl" deviceset="R-US_" device="R0805" value="120R"/>
 </parts>
 <sheets>
@@
 <instance part="RDIV2" gate="G$1" x="60.96" y="121.92" rot="R90"/>
 <instance part="RBOOT0" gate="G$1" x="-50.8" y="223.52" rot="R90"/>
+<instance part="RTERM" gate="G$1" x="121.92" y="182.88" rot="R180"/>
 </instances>
 <busses>
@@
 <pinref part="CAN" gate="-3" pin="KL"/>
 </segment>
+<segment>
+<pinref part="RTERM" gate="G$1" pin="2"/>
+<wire x1="111.76" y1="182.88" x2="116.84" y2="182.88" width="0.1524" layer="91"/>
+<label x="111.76" y="182.88" size="1.27" layer="95" rot="R180" xref="yes"/>
+</segment>
 </net>
 <net name="CANL" class="0">
@@
 <pinref part="CAN" gate="-1" pin="KL"/>
 </segment>
-</net>
+<segment>
+<pinref part="RTERM" gate="G$1" pin="1"/>
+<wire x1="132.08" y1="182.88" x2="127" y2="182.88" width="0.1524" layer="91"/>
+<label x="132.08" y="182.88" size="1.27" layer="95" xref="yes"/>
+</segment>
+</net>
