File: hw-demo02/hw-demo02.brd (EAGLE design)
At the start: 58.4 x 61 mm, 15 parts

Commit message: made the 12v pour a bit wider around the input connector
Routing:
- net +12V: vias 401 -> 412
Changed lines of the file:
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@@
 <signal name="+12V">
 <polygon width="0.4064" layer="1" spacing="0.3048" isolate="0.254" rank="4">
-<vertex x="46.0375" y="58.7375"/>
-<vertex x="46.0375" y="44.97605"/>
-<vertex x="47.83355" y="43.18"/>
+<vertex x="48.26" y="58.7375"/>
+<vertex x="48.26" y="44.97605"/>
+<vertex x="50.05605" y="43.18"/>
 <vertex x="57.4675" y="43.18"/>
 <vertex x="57.4675" y="5.464525"/>
@@
 <vertex x="57.4675" y="5.3975"/>
 <vertex x="57.4675" y="43.18"/>
-<vertex x="47.83355" y="43.18"/>
-<vertex x="46.0375" y="44.97605"/>
-<vertex x="46.0375" y="58.7375"/>
+<vertex x="50.05605" y="43.18"/>
+<vertex x="48.26" y="44.97605"/>
+<vertex x="48.26" y="58.7375"/>
 <vertex x="36.195" y="58.7375"/>
 <vertex x="36.195" y="38.735"/>
@@
 <vertex x="23.495" y="26.3525"/>
 </polygon>
+<via x="47.3075" y="58.1025" extent="1-16" drill="0.6"/>
+<via x="47.3075" y="56.515" extent="1-16" drill="0.6"/>
+<via x="47.3075" y="54.9275" extent="1-16" drill="0.6"/>
+<via x="47.3075" y="53.34" extent="1-16" drill="0.6"/>
+<via x="47.3075" y="51.7525" extent="1-16" drill="0.6"/>
+<via x="47.3075" y="50.165" extent="1-16" drill="0.6"/>
+<via x="47.3075" y="48.5775" extent="1-16" drill="0.6"/>
+<via x="47.3075" y="46.99" extent="1-16" drill="0.6"/>
+<via x="47.3075" y="45.4025" extent="1-16" drill="0.6"/>
+<via x="47.3075" y="43.815" extent="1-16" drill="0.6"/>
+<via x="48.895" y="43.815" extent="1-16" drill="0.6"/>
 </signal>
 <signal name="IN">
